Commit message: Small aesthetic changes to robot description files

File: urdf_example1/description/urdf/macros/wheel.xacro (robot description, xacro)
@@ -1,14 +1,15 @@
 <?xml version="1.0"?>
 <robot xmlns:xacro="http://ros.org/wiki/xacro">
-    <!--wheel params are: (distinctive part of) link name, 3d position, yaw angle, radius, thickness and mass-->
-    <xacro:macro name="wheel" params="name x:=0 y:=0 z:=0 ya:=0 wr:=^ wt:=^ wm:=^ gazebo:=^">
+    <!--wheel params are: (distinctive part of) link name, 3d position, radius, thickness and mass-->
+    <xacro:macro name="wheel" params="name x:=0 y:=0 z:=0 wr:=^ wt:=^ wm:=^ gazebo:=^">
         <joint name="base_to_${name}_wheel" type="continuous">
             <parent link="base_link"/>
             <child link="${name}_wheel"/>
-            <origin xyz="${x} ${y} ${z}" rpy="0 0 ${ya}"/>
+            <origin xyz="${x} ${y} ${z}"/>
+            <axis xyz="0 1 0"/>
         </joint>
         <link name="${name}_wheel">
             <visual>
-                <origin xyz="0 0 0" rpy="0 ${pi/2} 0"/>
+                <origin xyz="0 0 0" rpy="${pi/2} 0 0"/>
                 <geometry>
                     <cylinder length="${wt}" radius="${wr}"/>
@@ -17,5 +18,5 @@
             </visual>
             <collision>
-                <origin xyz="0 0 0" rpy="0 ${pi/2} 0"/>
+                <origin xyz="0 0 0" rpy="${pi/2} 0 0"/>
                 <geometry>
                     <cylinder length="${wt}" radius="${wr}"/>

File: urdf_example1/description/urdf/robot1.xacro (robot description, xacro)
@@ -6,4 +6,5 @@
     <xacro:include filename="$(find urdf_example1)/description/urdf/macros/base.xacro"/>
     <xacro:include filename="$(find urdf_example1)/description/urdf/macros/wheel.xacro"/>
+    <xacro:include filename="$(find urdf_example1)/description/urdf/macros/driving_plugin.xacro"/>
     <!--base dimensions (length, width and height) and mass-->
     <xacro:property name="bl" value="1"/>
@@ -18,26 +19,11 @@
     <xacro:base/>
     <!--create wheels-->
-    <xacro:wheel name="front_right" x="${bl/2-wr}" y="${-(bw+wt)/2}" ya="${pi/2}"/>
-    <xacro:wheel name="back_right" x="${-bl/2+wr}" y="${-(bw+wt)/2}" ya="${pi/2}"/>
-    <xacro:wheel name="back_left" x="${-bl/2+wr}" y="${(bw+wt)/2}" ya="${pi/2}"/>
-    <xacro:wheel name="front_left" x="${bl/2-wr}" y="${(bw+wt)/2}" ya="${pi/2}"/>
+    <xacro:wheel name="front_right" x="${bl/2-wr}" y="${-(bw+wt)/2}"/>
+    <xacro:wheel name="back_right" x="${-bl/2+wr}" y="${-(bw+wt)/2}"/>
+    <xacro:wheel name="back_left" x="${-bl/2+wr}" y="${(bw+wt)/2}"/>
+    <xacro:wheel name="front_left" x="${bl/2-wr}" y="${(bw+wt)/2}"/>
     <!--Add Gazebo driving plugin, if requested-->
     <xacro:if value="${gazebo}">
-        <gazebo>
-            <plugin name="skid_steer_drive_controller" filename="libgazebo_ros_skid_steer_drive.so">
-                <updateRate>50.0</updateRate>
-                <robotNamespace>/</robotNamespace>
-                <leftFrontJoint>base_to_front_left_wheel</leftFrontJoint>
-                <rightFrontJoint>base_to_front_right_wheel</rightFrontJoint>
-                <leftRearJoint>base_to_back_left_wheel</leftRearJoint>
-                <rightRearJoint>base_to_back_right_wheel</rightRearJoint>
-                <wheelSeparation>${bw+wt}</wheelSeparation>
-                <wheelDiameter>${2*wr}</wheelDiameter>
-                <robotBaseFrame>base_link</robotBaseFrame>
-                <torque>200</torque>
-                <topicName>cmd_vel</topicName>
-                <broadcastTF>true</broadcastTF>
-            </plugin>
-        </gazebo>
+        <xacro:skid_steer/>
     </xacro:if>
 </robot>
