Commit message: Add simple meshes

File: urdf_example1/description/urdf/macros/base.xacro (robot description, xacro)
@@ -7,6 +7,7 @@
                 <geometry>
                     <box size="${bl} ${bw} ${bh}"/>
+                    <!--<mesh filename="package://urdf_example1/description/meshes/fusca.stl" scale="${bl} ${bw} ${bh}"/>-->
                 </geometry>
-                <material name="red"/>
+                <material name="green"/>
             </visual>
             <collision>
@@ -23,5 +24,5 @@
         <xacro:if value="${gazebo}">
             <gazebo reference="base_link">
-                <material>Gazebo/Red</material>
+                <material>Gazebo/Green</material>
             </gazebo>
         </xacro:if>

File: urdf_example1/description/urdf/macros/wheel.xacro (robot description, xacro)
@@ -13,7 +13,8 @@
                 <origin xyz="0 0 0" rpy="${pi/2} 0 0"/>
                 <geometry>
-                    <cylinder length="${wt}" radius="${wr}"/>
+                    <!--<cylinder length="${wt}" radius="${wr}"/>-->
+                    <mesh filename="package://urdf_example1/description/meshes/monster_wheel.stl" scale="${2*wr} ${2*wr} ${wt}"/>
                 </geometry>
-                <material name="black"/>
+                <material name="gray"/>
             </visual>
             <collision>
@@ -35,5 +36,5 @@
                 <kp>1000000.0</kp>
                 <kd>1.0</kd>
-                <material>Gazebo/Black</material>
+                <material>Gazebo/Grey</material>
             </gazebo>
         </xacro:if>

Commit message: Fix fake joint_states being published and visualized in RVIZ

File: urdf_example1/description/urdf/macros/base.xacro (robot description, xacro)
@@ -21,5 +21,5 @@
             </inertial>
         </link>
-        <!--Add Gazebo references, if requested-->
+        <!--Add gazebo references, if requested-->
         <xacro:if value="${gazebo}">
             <gazebo reference="base_link">

File: urdf_example1/description/urdf/macros/gazebo_top_level_plugins.xacro (robot description, xacro)
@@ -1,21 +1,32 @@
 <?xml version="1.0"?>
 <robot xmlns:xacro="http://ros.org/wiki/xacro">
-    <xacro:macro name="skid_steer" params="bw:=^ wt:=^ wr:=^">
+    <xacro:macro name="joints_publisher">
+        <gazebo>
+            <plugin name="joint_state_publisher" filename="libgazebo_ros_joint_state_publisher.so">
+                <robotNamespace>/</robotNamespace>
+                <updateRate>50</updateRate>
+                <jointName>
+                    base_to_front_right_wheel, base_to_back_right_wheel, base_to_back_left_wheel, base_to_front_left_wheel
+                </jointName>
+            </plugin>
+        </gazebo>
+    </xacro:macro>
+    <xacro:macro name="skid_steer" params="bw:=^ wt:=^ wr:=^ tf_broadcast:=true">
         <gazebo>
             <plugin name="skid_steer_drive_controller" filename="libgazebo_ros_skid_steer_drive.so">
+                <robotNamespace>/</robotNamespace>
                 <updateRate>50.0</updateRate>
-                <robotNamespace>/</robotNamespace>
                 <commandTopic>cmd_vel</commandTopic>
                 <odometryTopic>odom</odometryTopic>
                 <robotBaseFrame>base_link</robotBaseFrame>
                 <odometryFrame>odom</odometryFrame>
-                <broadcastTF>true</broadcastTF>
+                <broadcastTF>${tf_broadcast}</broadcastTF> <!--only odom to base_link-->
+                <rightFrontJoint>base_to_front_right_wheel</rightFrontJoint>
+                <rightRearJoint>base_to_back_right_wheel</rightRearJoint>
+                <leftRearJoint>base_to_back_left_wheel</leftRearJoint>
                 <leftFrontJoint>base_to_front_left_wheel</leftFrontJoint>
-                <rightFrontJoint>base_to_front_right_wheel</rightFrontJoint>
-                <leftRearJoint>base_to_back_left_wheel</leftRearJoint>
-                <rightRearJoint>base_to_back_right_wheel</rightRearJoint>
                 <wheelSeparation>${bw+wt}</wheelSeparation>
                 <wheelDiameter>${2*wr}</wheelDiameter>
-                <torque>200</torque>
+                <torque>100</torque>
                 <covariance_x>0.0001</covariance_x>
                 <covariance_y>0.0001</covariance_y>

File: urdf_example1/description/urdf/macros/wheel.xacro (robot description, xacro)
@@ -29,5 +29,5 @@
             </inertial>
         </link>
-        <!--Add Gazebo references, if requested-->
+        <!--Add gazebo references, if requested-->
         <xacro:if value="${gazebo}">
             <gazebo reference="${name}_wheel">

File: urdf_example1/description/urdf/robot1.xacro (robot description, xacro)
@@ -6,5 +6,5 @@
     <xacro:include filename="$(find urdf_example1)/description/urdf/macros/base.xacro"/>
     <xacro:include filename="$(find urdf_example1)/description/urdf/macros/wheel.xacro"/>
-    <xacro:include filename="$(find urdf_example1)/description/urdf/macros/driving_plugin.xacro"/>
+    <xacro:include filename="$(find urdf_example1)/description/urdf/macros/gazebo_top_level_plugins.xacro"/>
     <!--base dimensions (length, width and height) and mass-->
     <xacro:property name="bl" value="1"/>
@@ -23,6 +23,7 @@
     <xacro:wheel name="back_left" x="${-bl/2+wr}" y="${(bw+wt)/2}"/>
     <xacro:wheel name="front_left" x="${bl/2-wr}" y="${(bw+wt)/2}"/>
-    <!--Add Gazebo driving plugin, if requested-->
+    <!--Add gazebo plugins, if requested-->
     <xacro:if value="${gazebo}">
+        <xacro:joints_publisher/>
         <xacro:skid_steer/>
     </xacro:if>
