Commit message: Add a new robot with multiple laser scanners

File: urdf_example1/description/urdf/macros/laser_scanners.xacro (robot description, xacro)
@@ -1,14 +1,14 @@
 <?xml version="1.0"?>
 <robot xmlns:xacro="http://ros.org/wiki/xacro">
-    <!--wheel params are: laser name, 3d position, orientation and a gazebo flag-->
+    <!--URG-04LX-UG01-->
     <xacro:macro name="hokuyo" params="name xyz rpy gazebo:=^">
         <joint name="base_to_${name}" type="fixed">
             <parent link="base_link"/>
             <child link="${name}"/>
-            <origin xyz="${xyz}"/>
+            <origin xyz="${xyz}" rpy="${rpy}"/>
         </joint>
         <link name="${name}">
             <visual>
-                <origin xyz="0 0 0" rpy="${rpy}"/>
+                <origin xyz="0 0 0" rpy="0 0 0"/>
                 <geometry>
                     <mesh filename="package://urdf_example1/description/meshes/hokuyo.dae"/>
@@ -16,5 +16,5 @@
             </visual>
             <collision>
-                <origin xyz="0 0 0" rpy="${rpy}"/>
+                <origin xyz="0 0 0" rpy="0 0 0"/>
                 <geometry>
                     <box size="0.1 0.1 0.1"/>
@@ -29,20 +29,19 @@
         <xacro:if value="${gazebo}">
             <gazebo reference="${name}">
-                <sensor type="gpu_ray" name="${name}_sensor">
+                <sensor name="${name}_sensor" type="gpu_ray">
                     <pose>0 0 0 0 0 0</pose>
+                    <update_rate>10</update_rate>
                     <visualize>true</visualize>
-                    <update_rate>40</update_rate>
                     <ray>
                         <scan>
                             <horizontal>
-                                <samples>720</samples>
-                                <resolution>1</resolution>
-                                <min_angle>-1.570796</min_angle>
-                                <max_angle>1.570796</max_angle>
+                                <samples>683</samples>
+                                <min_angle>${-2*pi/3}</min_angle>
+                                <max_angle>${2*pi/3}</max_angle>
                             </horizontal>
                         </scan>
                         <range>
-                            <min>0.10</min>
-                            <max>4.0</max>
+                            <min>0.02</min>
+                            <max>5.6</max>
                             <resolution>0.01</resolution>
                         </range>
@@ -50,10 +49,11 @@
                             <type>gaussian</type>
                             <mean>0.0</mean>
-                            <stddev>0.01</stddev>
+                            <stddev>0.05</stddev>
                         </noise>
                     </ray>
                     <plugin name="${name}_plugin" filename="libgazebo_ros_gpu_laser.so">
+                        <robotNamespace>/</robotNamespace>
+                        <frameName>${name}</frameName>
                         <topicName>${name}</topicName>
-                        <frameName>${name}</frameName>
                     </plugin>
                 </sensor>

File: urdf_example1/description/urdf/robot3.xacro (robot description, xacro)
@@ -26,4 +26,5 @@
     <!--Add laser scanners-->
     <xacro:hokuyo name="front_scan" xyz="${bl/2-0.05} 0 ${bh/2+0.05}" rpy="0 0 0"/>
+    <xacro:hokuyo name="back_scan" xyz="${-bl/2+0.05} 0 ${bh/2+0.05}" rpy="0 0 ${pi}"/>
     <!--Add top-level gazebo plugins, if requested-->
     <xacro:if value="${gazebo}">

Commit message: Add new lms200 laser scanner option

File: urdf_example1/description/urdf/macros/laser_scanners.xacro (robot description, xacro)
@@ -1,5 +1,6 @@
 <?xml version="1.0"?>
 <robot xmlns:xacro="http://ros.org/wiki/xacro">
-    <!--URG-04LX-UG01-->
+    <!--hokuyo URG-04LX-UG01 laser scanner-->
+    <!--Parameters are: link/frame name, position, orientation and gazebo flag-->
     <xacro:macro name="hokuyo" params="name xyz rpy gazebo:=^">
         <joint name="base_to_${name}" type="fixed">
@@ -32,5 +33,5 @@
                     <pose>0 0 0 0 0 0</pose>
                     <update_rate>10</update_rate>
-                    <visualize>true</visualize>
+                    <visualize>false</visualize>
                     <ray>
                         <scan>
@@ -43,5 +44,6 @@
                         <range>
                             <min>0.02</min>
-                            <max>5.6</max>
+                            <!--should be 5.6, but gazebo exhibits weird behaviour for 5.7 or smaller ???-->
+                            <max>5.8</max>
                             <resolution>0.01</resolution>
                         </range>
@@ -61,3 +63,64 @@
         </xacro:if>
     </xacro:macro>
+    <!--SICK LMS-200 laser scanner-->
+    <!--Parameters are: link/frame name, position, orientation and gazebo flag-->
+    <xacro:macro name="lms200" params="name xyz rpy gazebo:=^">
+        <joint name="base_to_${name}" type="fixed">
+            <parent link="base_link"/>
+            <child link="${name}"/>
+            <origin xyz="${xyz}" rpy="${rpy}"/>
+        </joint>
+        <link name="${name}">
+            <visual>
+                <origin xyz="0 0 0" rpy="0 0 0"/>
+                <geometry>
+                    <mesh filename="package://urdf_example1/description/meshes/lms200.dae"/>
+                </geometry>
+            </visual>
+            <collision>
+                <origin xyz="0 0 0" rpy="0 0 0"/>
+                <geometry>
+                    <box size="0.156 0.155 0.185"/>
+                </geometry>
+            </collision>
+            <inertial>
+                <mass value="1e-5" />
+                <inertia ixx="1e-6" ixy="0" ixz="0" iyy="1e-6" iyz="0" izz="1e-6" />
+            </inertial>
+        </link>
+        <!--Add gazebo references, if requested-->
+        <xacro:if value="${gazebo}">
+            <gazebo reference="${name}">
+                <sensor name="${name}_sensor" type="gpu_ray">
+                    <pose>0 0 0 0 0 0</pose>
+                    <update_rate>75</update_rate>
+                    <visualize>false</visualize>
+                    <ray>
+                        <scan>
+                            <horizontal>
+                                <samples>361</samples>
+                                <min_angle>${-pi/2}</min_angle>
+                                <max_angle>${pi/2}</max_angle>
+                            </horizontal>
+                        </scan>
+                        <range>
+                            <min>0.02</min>
+                            <max>10.0</max>
+                            <resolution>0.01</resolution>
+                        </range>
+                        <noise>
+                            <type>gaussian</type>
+                            <mean>0.0</mean>
+                            <stddev>0.015</stddev>
+                        </noise>
+                    </ray>
+                    <plugin name="${name}_plugin" filename="libgazebo_ros_gpu_laser.so">
+                        <robotNamespace>/</robotNamespace>
+                        <frameName>${name}</frameName>
+                        <topicName>${name}</topicName>
+                    </plugin>
+                </sensor>
+            </gazebo>
+        </xacro:if>
+    </xacro:macro>
 </robot>

File: urdf_example1/description/urdf/robot3.xacro (robot description, xacro)
@@ -1,4 +1,4 @@
 <?xml version="1.0"?>
-<robot name="robot2" xmlns:xacro="http://ros.org/wiki/xacro">
+<robot name="robot3" xmlns:xacro="http://ros.org/wiki/xacro">
     <xacro:arg name="gazebo" default="false"/>
     <xacro:property name="gazebo" value="$(arg gazebo)"/>

Commit message: Change name of xacro macro of lms200 laser scanner

File: urdf_example1/description/urdf/macros/laser_scanners.xacro (robot description, xacro)
@@ -65,5 +65,5 @@
     <!--SICK LMS-200 laser scanner-->
     <!--Parameters are: link/frame name, position, orientation and gazebo flag-->
-    <xacro:macro name="lms200" params="name xyz rpy gazebo:=^">
+    <xacro:macro name="sick" params="name xyz rpy gazebo:=^">
         <joint name="base_to_${name}" type="fixed">
             <parent link="base_link"/>
